File: hardware/KiCad/BodyTempSensor.kicad_sch (KiCad schematic)
At the start: 84 parts, among them IC3 TMP117MAIDRVR, IC4 TMP117MAIDRVT, IC5 TMP117MAIDRVT, IC6 TMP117MAIDRVT, IC7 NRF54L15-QFAA-R, J1 USB_C_Receptacle_USB2.0, J3 BAT, J6 Conn_02x05_Odd_Even, Q1 NMOS, Q2 NMOS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

Commit message: Updated KiCad and BOM
Parts:
- removed C26: 100n, Capacitor_SMD:C_0402_1005Metric_Pad0.74x0.62mm_HandSolder, symbol Device:C
- C1: Manufacturer_Name KDS Daishinku -> YAGEO
- C13: value 100n -> 2n2; LCSC PART # C361203 -> C106861; Manufacturer_Part_Number C1005X5R1E104KT000E -> CC0402KRX7R9BB222
- C18: LCSC PART # (none) -> C7393858; Manufacturer_Name (none) -> CCTC; Manufacturer_Part_Number (none) -> TCC0402X5R394K160AT
- C2: footprint Capacitor_SMD:C_0504_1310Metric_Pad0.83x1.28mm_HandSolder -> Capacitor_SMD:C_0402_1005Metric_Pad0.74x0.62mm_HandSolder; LCSC PART # (none) -> C106254; Manufacturer_Name (none) -> YAGEO; Manufacturer_Part_Number (none) -> CC0402KRX5R6BB105
- C27: LCSC PART # (none) -> C327025; Manufacturer_Name (none) -> YAGEO; Manufacturer_Part_Number (none) -> CC0402KRX7R8BB103
- C28, C30: LCSC PART # (none) -> C295941; Manufacturer_Name (none) -> Walsin Tech Corp; Manufacturer_Part_Number (none) -> 0402X225K100CT
- C29: LCSC PART # (none) -> C106861; Manufacturer_Name (none) -> YAGEO; Manufacturer_Part_Number (none) -> CC0402KRX7R9BB222
- C4: LCSC PART # (none) -> TBT
- C6, C9: LCSC PART # (none) -> C106201; Manufacturer_Name (none) -> YAGEO; Manufacturer_Part_Number (none) -> CC0402JRNPO9BN120
- C8: LCSC PART # (none) -> CC0402BRNPO9BN2R0; Manufacturer_Name (none) -> YAGEO; Manufacturer_Part_Number (none) -> CC0402BRNPO9BN2R0
- D1, D2, D3: footprint LED_SMD:LED_0603_1608Metric_Pad1.05x0.95mm_HandSolder -> LED_SMD:LED_0402_1005Metric_Pad0.77x0.64mm_HandSolder; LCSC PART # (none) -> C965790; Manufacturer_Name (none) -> XINGLIGHT; Manufacturer_Part_Number (none) -> XL-1005SURC
- H1, H2: value MountingHole_Pad -> (none); footprint MountingHole:MountingHole_2.2mm_M2_DIN965_Pad -> (none)
- IC3: value TMP117MAIDRVR -> TMP117MAIDRVT; footprint LibLoader:SON65P200X200X80-7N -> PCB_Lib_ItsNotDaan:SON65P200X200X80-7N; LCSC PART # (none) -> C2803242; Manufacturer_Part_Number TMP117MAIDRVT -> TMP117MAIDRVR
- IC4, IC5, IC6: footprint LibLoader:SON65P200X200X80-7N -> PCB_Lib_ItsNotDaan:SON65P200X200X80-7N; LCSC PART # (none) -> C2803242; Manufacturer_Part_Number TMP117MAIDRVT -> TMP117MAIDRVR
- IC7: footprint LibLoader:QFN40P600X600X95-49N -> PCB_Lib_ItsNotDaan:QFN40P600X600X95-49N; LCSC PART # (none) -> C42458750
- J1: footprint Connector_USB:USB_C_Receptacle_GCT_USB4105-xx-A_16P_TopMnt_Horizontal -> PCB_Lib_ItsNotDaan:USB_C_Receptacle_GCT_USB4105-xx-A_16P_TopMnt_Horizontal; LCSC PART # (none) -> C223907; Manufacturer_Name (none) -> Korean Hroparts Elec; Manufacturer_Part_Number (none) -> TYPE-C-31-M-14
- L1, L4: value 3.5nH -> 3n5; footprint Inductor_SMD:L_0201_0603Metric -> Inductor_SMD:L_0201_0603Metric_Pad0.64x0.40mm_HandSolder; LCSC PART # (none) -> C52109755; Manufacturer_Name (none) -> CCTC; Manufacturer_Part_Number LQP03HQ3N5B02 -> TCGL0603C3N5SZT
- L3: value 2.7nH -> 2n7; footprint Inductor_SMD:L_0201_0603Metric -> Inductor_SMD:L_0402_1005Metric_Pad0.77x0.64mm_HandSolder; LCSC PART # (none) -> C77108; Manufacturer_Name (none) -> muRata; Manufacturer_Part_Number LQP03HQ2N7B02 -> LQG15HS2N7S02D
- L5: footprint Inductor_SMD:L_0201_0603Metric -> Inductor_SMD:L_0603_1608Metric_Pad1.05x0.95mm_HandSolder; LCSC PART # (none) -> C76799; Manufacturer_Name (none) -> TDK; Manufacturer_Part_Number (none) -> MLZ1608M4R7WT000
- Q1, Q2: footprint (none) -> Package_TO_SOT_SMD:SOT-23; LCSC PART # (none) -> C20917; Manufacturer_Name (none) -> AOS; Manufacturer_Part_Number (none) -> AO3400A
- R1, R2, R26, R27: LCSC PART # (none) -> C105873; Manufacturer_Name (none) -> YAGEO; Manufacturer_Part_Number (none) -> RC0402JR-075K1L
- R11: LCSC PART # (none) -> C238338; Manufacturer_Name (none) -> YAGEO; Manufacturer_Part_Number (none) -> RC0402FR-0768KL
- R17: LCSC PART # (none) -> C137932; Manufacturer_Name (none) -> YAGEO; Manufacturer_Part_Number (none) -> RC0402FR-0782KL
- R21, R23, R28: LCSC PART # (none) -> C138046; Manufacturer_Name (none) -> YAGEO; Manufacturer_Part_Number (none) -> RC0402FR-07180KL
- R22: LCSC PART # (none) -> C93943; Manufacturer_Name (none) -> YAGEO; Manufacturer_Part_Number (none) -> RC0402FR-0747KL
- R4, R5, R6: LCSC PART # (none) -> C3017744; Manufacturer_Name (none) -> VO; Manufacturer_Part_Number (none) -> SCR0603J470R
- R7: value 10k -> 450k; LCSC PART # C163810 -> C5159688; Manufacturer_Name Walsin Tech Corp -> FOJAN; Manufacturer_Part_Number WR04X1002FTL -> FRC0402F4503TS
- R9: LCSC PART # (none) -> C106235; Manufacturer_Name (none) -> YAGEO; Manufacturer_Part_Number (none) -> RC0402FR-071KL
- RST1: value SW_RST -> MCP73833-xxx-UN; footprint PCB_Lib_ItsNotDaan:SW_SPST_EVQP2 -> Package_SO:MSOP-10_3x3mm_P0.5mm; LCSC PART # C512395 -> C424093; Manufacturer_Name PANASONIC -> MICROCHIP; Manufacturer_Part_Number EVQP2P02W -> MCP73831T-2ACI/OT
- U2: LCSC PART # (none) -> C2827654; Manufacturer_Name (none) -> TECH PUBLIC; Manufacturer_Part_Number (none) -> USBLC6-2SC6
- U3: LCSC PART # (none) -> C424093; Manufacturer_Name (none) -> MICROCHIP; Manufacturer_Part_Number (none) -> MCP73831T-2ACI/OT
- U5: LCSC PART # (none) -> C116490; Manufacturer_Name (none) -> Microchip; Manufacturer_Part_Number (none) -> MCP6001T-I/OT
- Y1: LCSC PART # (none) -> C113671; Manufacturer_Name (none) -> YXC; Manufacturer_Part_Number (none) -> X322532MMB4SI
Connections:
- net +3V3: now also C11.1
- net VBUS: no longer C11.1
Other:
- moved on the sheet: C11, TP1
