File: hardware/KiCad/BodyTempSensor.kicad_pcb (KiCad board)
At the start: 4 copper layers, 80 x 35 mm, 80 parts, among them IC3 TMP117MAIDRVT, IC4 TMP117MAIDRVT, IC5 TMP117MAIDRVT, IC6 TMP117MAIDRVT, IC7 NRF54L15-QFAA-R, J1 USB_C_Receptacle_USB2.0, J3 BAT, J6 Conn_02x05_Odd_Even, Q1 NMOS, Q2 NMOS, U2 USBLC6-2SC6, U3 MCP73833-xxx-UN, U4 TLV62568DBVR, U5 MCP6001-OT, Y1 32MHz

Commit message: Did 80% of the PCB lay-out
Parts:
- removed U2: USBLC6-2SC6, Package_TO_SOT_SMD:SOT-23-6
- TP3, TP4: moved to B.Cu
- moved H1 50.2 mm to (184.7, 103.8), turned to 180 degrees
- moved H2 49.7 mm to (184.7, 93.8), turned to 180 degrees
- moved Q1 41.9 mm to (200.5, 112.1)
- moved R11 39.8 mm to (184.7, 107.5)
- moved R13 27.9 mm to (195.9, 108.9), turned to 180 degrees
- moved U5 27.3 mm to (192.0, 109.9)
- moved C18 27.3 mm to (191.3, 106.4)
- moved R17 27.3 mm to (191.3, 107.5)
- moved R14 26.9 mm to (195.9, 110.0), turned to 0 degrees
- moved C12 26.6 mm to (184.2, 111.1), turned to 0 degrees
- moved R20 26.2 mm to (199.7, 115.5), turned to 180 degrees
- moved J6 26.2 mm to (175.5, 114.9), turned to 90 degrees
- moved TP2 25.8 mm to (185.2, 114.0), turned to 0 degrees
- moved LED1 25.8 mm to (185.2, 114.0)
- moved R21 23.2 mm to (199.7, 114.5)
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Connections:
- J1 pad A6: /USB_D+ -> unconnected-(J1-D+-PadA6)
- J1 pad A7: /USB_D- -> unconnected-(J1-D--PadA7)
- J1 pad B6: /USB_D+ -> unconnected-(J1-D+-PadB6)
- J1 pad B7: /USB_D- -> unconnected-(J1-D--PadB7)
Routing:
- net VBAT: track 35.6 -> 10.5 mm, vias 0 -> 2
- net Earth: track 8.00 -> 30.4 mm, vias 0 -> 32
- net /USB_D+: track 8.11 -> 0.00 mm
- net /USB_D-: track 8.05 -> 0.00 mm
- net +3V3: track 28.6 -> 23.0 mm, vias 0 -> 16
- net Net-(U4-SW): track 5.48 -> 0.00 mm
- net /AMP_1: track 0.00 -> 4.39 mm
- net Net-(IC7A-DECA): track 0.00 -> 3.62 mm
- net VBUS: track 3.86 -> 0.50 mm
- net Net-(H1-Pad1): track 0.00 -> 3.08 mm
- net Net-(U3-STAT2): track 0.00 -> 2.74 mm
- net Net-(Q1-G): track 0.00 -> 2.70 mm
- net Net-(U5--): track 0.00 -> 2.58 mm
- net Net-(U3-STAT1): track 0.00 -> 2.15 mm
- net Net-(Q1-D): track 0.00 -> 1.60 mm
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- added copper zone on F.Cu, net +3V3
- added copper zone on In2.Cu, net +3V3
- added copper zone on In1.Cu, net Earth
- added copper zone on F.Cu, net Net-(U4-SW)
- added copper zone on In2.Cu, net VBAT
- added copper zone on In2.Cu, net VBUS
Other:
- outline, holes or cut-outs redrawn
- board text added: "+"
- board text added: "-"
- board text added: "3V3 Buck"
- board text added: "ANT"
- board text added: "Bat Chr"
- board text added: "Bat Meas"
- board text added: "Button"
- board text added: "DIO,SWD,XXX,XXX,RST 3V3,GND,GND,XXX,XXX"
- board text added: "JTAG"
- board text added: "MCU NRF54L15"
- board text added: "RGB"
- board text added: "Res Meas"
- board text added: "USB CHRG"
